Commit message: Camera node

File: assets/robot/r1_pro/r1_pro.urdf (robot description, URDF)
Before this commit: robot r1_pro, 46 links, 45 joints
Links:
- added link t265_link, mass 0.068024; collision mesh filename=meshes/t265.stl; visual mesh filename=meshes/t265.stl
- added link t265_mount; collision mesh filename=meshes/t265_mount.stl; visual mesh filename=meshes/t265_mount.stl
- added link t265_pose_tracking_frame
Joints:
- added joint t265_joint: type fixed, parent t265_mount, child t265_link, origin xyz=-0.017454 -0.000393 0.000262 rpy=1.57079632679 0 1.57079632679, axis 0 0 0
- added joint t265_mount_joint: type fixed, parent base_link, child t265_mount, origin xyz=-0.217664 0 0.31299 rpy=0 0 0, axis 0 0 0
- added joint t265_pose_tracking_joint: type fixed, parent t265_link, child t265_pose_tracking_frame, origin xyz=-0.0091 0.0 0.0 rpy=-1.57079632679 1.57079632679 0
